Commit message: Update files

File: src/my_robot/urdf/my_robot.xacro (robot description, xacro)
@@ -55,5 +55,8 @@
                                                     </visual>
                                                   </link>
-                                                                                                     <link name="left_wheel">
+                                                  <gazebo reference="chassis">
+							    <material>Gazebo/Blue</material>
+						</gazebo>
+                                                  <link name="left_wheel">
                                                     <inertial>
                                                       <mass value="5.0"/>
@@ -71,5 +74,5 @@
                                                       </geometry>
                                                     </collision>
-                                                    <visual name='chassis_visual'>
+                                                    <visual name='left_wheel_visual'>
                                                       <origin xyz="0.0 0 0" rpy="0 1.5707 1.5707"/>
                                                       <geometry>
@@ -78,4 +81,7 @@
                                                     </visual>
                                                     </link>
+                                                    	<gazebo reference="left_wheel">
+							    <material>Gazebo/Green</material>
+							</gazebo>
                                                     <joint type="continuous" name="left_wheel_hinge">
 							    <origin xyz="0 0.15 0" rpy="0 0 0"/>
@@ -102,5 +108,5 @@
                                                       </geometry>
                                                     </collision>
-                                                    <visual name='chassis_visual'>
+                                                    <visual name='right_wheel_visual'>
                                                       <origin xyz="0.0 0 0" rpy="0 1.5707 1.5707"/>
                                                       <geometry>
@@ -109,5 +115,8 @@
                                                     </visual>
                                                     </link>
-                                                    <joint type="continuous" name="right_wheel_hingo">
+                                                    <gazebo reference="right_wheel">
+							    <material>Gazebo/Green</material>
+							</gazebo>
+                                                    <joint type="continuous" name="right_wheel_hinge">
 							    <origin xyz="0 -0.15 0" rpy="0 0 0"/>
 							    <child link="right_wheel"/>
@@ -117,3 +126,65 @@
 							    <dynamics damping="1.0" friction="1.0"/>
 							  </joint>
+	<link name="camera">
+		<inertial>
+			<mass value="0.1"/>
+			<origin xyz="0.0 0 0" rpy="0 0 0"/>
+			<inertia
+			ixx="1e-6" ixy="0" ixz="0"
+			iyy="1e-6" iyz="0"
+			izz="1e-6"
+			/>
+		</inertial>
+		<collision name='collision'>
+			<origin xyz="0.0 0 0" rpy="0 0 0"/>
+			<geometry>
+			<box size=".05 .05 .05"/>
+			</geometry>
+		</collision>
+		<visual name='camera_visual'>
+			<origin xyz="0.0 0 0" rpy="0 0 0"/>
+			<geometry>
+			<box size=".05 .05 .05"/>
+			</geometry>
+		</visual>
+	</link>
+	<gazebo reference="camera">
+	    <material>Gazebo/Red</material>
+	</gazebo>
+	<joint type="fixed" name="camera_joint">
+		<origin xyz="0.2 0 0" rpy="0 0 0"/>
+		<child link="camera"/>
+		<parent link="chassis"/>
+		<axis xyz="0 1 0" rpy="0 0 0"/>
+	</joint>
+	<link name="hokuyo">
+		<inertial>
+			<mass value="1e-5"/>
+			<origin xyz="0.0 0 0" rpy="0 0 0"/>
+			<inertia
+			ixx="1e-6" ixy="0" ixz="0"
+			iyy="1e-6" iyz="0"
+			izz="1e-6"
+			/>
+		</inertial>
+		<collision name='collision'>
+			<origin xyz="0.0 0 0" rpy="0 0 0"/>
+			<geometry>
+				<box size=".1 .1 .1"/>
+			</geometry>
+		</collision>
+		<visual name='visual'>
+			<origin xyz="0.0 0 0" rpy="0 0 0"/>
+			<geometry>
+				<mesh  filename = "package://my_robot/meshes/hokuyo.dae"/>
+			</geometry>
+		</visual>
+	</link>
+	<joint type="fixed" name="hokuyo_joint">
+		<origin xyz="0.15 0 0.1" rpy="0 0 0"/>
+		<child link="hokuyo"/>
+		<parent link="chassis"/>
+		<axis xyz="0 1 0" rpy="0 0 0"/>
+	</joint>
+  	<xacro:include filename="$(find my_robot)/urdf/my_robot.gazebo" />
 </robot>
